Commit message: Update diffbot.ros2_control.xacro

File: description/ros2_control/diffbot.ros2_control.xacro (robot description, xacro)
@@ -1,10 +1,12 @@
 <?xml version="1.0"?>
 <robot xmlns:xacro="http://www.ros.org/wiki/xacro">
-  <xacro:macro name="diffbot_ros2_control" params="name prefix">
+  <xacro:macro name="mechanumbot_ros2_control" params="name prefix">
     <ros2_control name="${name}" type="system">
       <hardware>
-        <plugin>diffdrive_arduino/DiffDriveArduinoHardware</plugin>
-        <param name="left_wheel_name">left_wheel_joint</param>
-        <param name="right_wheel_name">right_wheel_joint</param>
+        <plugin>mechanumdrive_arduino/MechanumDriveArduinoHardware</plugin>
+        <param name="front_left_wheel_name">${prefix}front_left_wheel_joint</param>
+        <param name="front_right_wheel_name">${prefix}front_right_wheel_joint</param>
+        <param name="rear_left_wheel_name">${prefix}rear_left_wheel_joint</param>
+        <param name="rear_right_wheel_name">${prefix}rear_right_wheel_joint</param>
         <param name="loop_rate">30</param>
         <param name="device">/dev/serial/by-path/platform-fd500000.pcie-pci-0000:01:00.0-usb-0:1.3:1.0-port0</param>
@@ -17,10 +19,20 @@
         <param name="pid_o">50</param>
       </hardware>
-      <joint name="${prefix}left_wheel_joint">
+      <joint name="${prefix}front_left_wheel_joint">
         <command_interface name="velocity"/>
         <state_interface name="position"/>
         <state_interface name="velocity"/>
       </joint>
-      <joint name="${prefix}right_wheel_joint">
+      <joint name="${prefix}front_right_wheel_joint">
+        <command_interface name="velocity"/>
+        <state_interface name="position"/>
+        <state_interface name="velocity"/>
+      </joint>
+      <joint name="${prefix}rear_left_wheel_joint">
+        <command_interface name="velocity"/>
+        <state_interface name="position"/>
+        <state_interface name="velocity"/>
+      </joint>
+      <joint name="${prefix}rear_right_wheel_joint">
         <command_interface name="velocity"/>
         <state_interface name="position"/>
